File: kicad/bookmark/project.kicad_pcb (KiCad board)
At the start: 2 copper layers, 27 x 177 mm, 53 parts, among them SW1 SW_DIP_x01

Commit message: fix: correct LED footprints
Parts:
- D1, D10, D11, D12, D13, D14, D15, D16, D17, D18, D19, D2, D20, D21, D22, D23, D24, D3, D4, D5, D6, D7, D8, D9: footprint custom-footprints:LED_SK6812_SIDE-A-S -> custom-footprints:LED-SMD_4P-L4.0-W1.6-L
- moved D1 0.51 mm to (51.0, 28.1)
- moved D10 0.51 mm to (51.0, 91.1)
- moved D11 0.51 mm to (51.0, 98.1)
- moved D12 0.51 mm to (51.0, 105.1)
- moved D13 0.51 mm to (51.0, 112.1)
- moved D14 0.51 mm to (51.0, 119.1)
- moved D15 0.51 mm to (51.0, 126.1)
- moved D16 0.51 mm to (51.0, 133.1)
- moved D17 0.51 mm to (51.0, 140.1)
- moved D18 0.51 mm to (51.0, 147.1)
- moved D19 0.51 mm to (51.0, 154.1)
- moved D2 0.51 mm to (51.0, 35.1)
- moved D20 0.51 mm to (51.0, 161.1)
- moved D21 0.51 mm to (51.0, 168.1)
- moved D22 0.51 mm to (51.0, 175.1)
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