File: kicad/bookmark/project.kicad_sch (KiCad schematic)
At the start: 53 parts, among them SW1 SW_DIP_x01

Commit message: fix: correct LED footprints
Parts:
- D1, D10, D11, D12, D13, D14, D15, D16, D17, D18, D19, D2, D20, D21, D22, D23, D24, D3, D4, D5, D6, D7, D8, D9: footprint custom-footprints:LED_SK6812_SIDE-A-S -> custom-footprints:LED-SMD_4P-L4.0-W1.6-L

Commit message: fix(bookmark): change 22uF value to 100uF cheapo. controller only uses 100uF and 0.1uF
Parts:
- C1: value 22u -> 100u
Changed lines of the file:
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@@
 			)
 		)
-		(property "Value" "22u"
+		(property "Value" "100u"
 			(at 36.068 28.702 0)
 			(show_name no)
